File: kicad5/smart-temp-only-sensor3/smart-temp-only-sensor3.sch (KiCad schematic (older format))
At the start: 2 parts, among them J1 USB_B_Mini, J2 Conn_01x04_Female

Commit message: noid: autoroute final beta
Parts:
- J1: footprint Connector_USB:USB_A_Molex_67643_Horizontal -> Connector_USB:USB_Mini-B_Tensility_54-00023_Vertical
- J2: footprint Connector_PinHeader_2.54mm:PinHeader_1x04_P2.54mm_Vertical -> Connector_PinSocket_2.54mm:PinSocket_1x04_P2.54mm_Vertical
Connections:
- net labels added: +3.3V, GND1
Other:
- moved on the sheet: J1
Changed lines of the file:
@@
 Comment4 ""
 $EndDescr
+NoConn ~ 5650 2600
+NoConn ~ 5250 2800
 $Comp
-L Connector:Conn_01x04_Female J2
-U 1 1 6339AE0F
-P 6151 2450
-F 0 "J2" H 6179 2426 50  0000 L CNN
-F 1 "Conn_01x04_Female" H 6179 2335 50  0000 L CNN
-F 2 "Connector_PinHeader_2.54mm:PinHeader_1x04_P2.54mm_Vertical" H 6151 2450 50  0001 C CNN
-F 3 "~" H 6151 2450 50  0001 C CNN
-	1    6151 2450
+L power:+3.3V #PWR0101
+U 1 1 633B9908
+P 6275 2150
+F 0 "#PWR0101" H 6275 2000 50  0001 C CNN
+F 1 "+3.3V" H 6290 2323 50  0000 C CNN
+F 2 "" H 6275 2150 50  0001 C CNN
+F 3 "" H 6275 2150 50  0001 C CNN
+	1    6275 2150
+	1    0    0    -1
+$EndComp
+$Comp
+L power:GND1 #PWR0104
+U 1 1 633BE5C3
+P 6275 2775
+F 0 "#PWR0104" H 6275 2525 50  0001 C CNN
+F 1 "GND1" H 6280 2602 50  0000 C CNN
+F 2 "" H 6275 2775 50  0001 C CNN
+F 3 "" H 6275 2775 50  0001 C CNN
+	1    6275 2775
 	1    0    0    -1
 $EndComp
@@
 L Connector:USB_B_Mini J1
 U 1 1 6339C102
-P 5150 2550
-F 0 "J1" H 5207 3017 50  0000 C CNN
-F 1 "USB_B_Mini" H 5207 2926 50  0000 C CNN
-F 2 "Connector_USB:USB_A_Molex_67643_Horizontal" H 5300 2500 50  0001 C CNN
-F 3 "~" H 5300 2500 50  0001 C CNN
-	1    5150 2550
+P 5350 2400
+F 0 "J1" H 5407 2867 50  0000 C CNN
+F 1 "USB_B_Mini" H 5407 2776 50  0000 C CNN
+F 2 "Connector_USB:USB_Mini-B_Tensility_54-00023_Vertical" H 5500 2350 50  0001 C CNN
+F 3 "~" H 5500 2350 50  0001 C CNN
+	1    5350 2400
+	1    0    0    -1
+$EndComp
+$Comp
+L Connector:Conn_01x04_Female J2
+U 1 1 633D28B1
+P 6475 2400
+F 0 "J2" H 6503 2376 50  0000 L CNN
+F 1 "Conn_01x04_Female" H 6503 2285 50  0000 L CNN
+F 2 "Connector_PinSocket_2.54mm:PinSocket_1x04_P2.54mm_Vertical" H 6475 2400 50  0001 C CNN
+F 3 "~" H 6475 2400 50  0001 C CNN
+	1    6475 2400
 	1    0    0    -1
 $EndComp
 Wire Wire Line
-	5950 2350 5450 2350
+	6275 2300 6275 2150
 Wire Wire Line
-	5950 2450 5745 2450
+	6275 2400 5650 2400
 Wire Wire Line
-	5745 2450 5745 2650
+	5650 2500 6275 2500
 Wire Wire Line
-	5950 2550 5450 2550
+	6275 2600 6275 2775
+$Comp
+L power:+3.3V #PWR0102
+U 1 1 633E08FC
+P 5800 2125
+F 0 "#PWR0102" H 5800 1975 50  0001 C CNN
+F 1 "+3.3V" H 5815 2298 50  0000 C CNN
+F 2 "" H 5800 2125 50  0001 C CNN
+F 3 "" H 5800 2125 50  0001 C CNN
+	1    5800 2125
+	1    0    0    -1
+$EndComp
 Wire Wire Line
-	5950 2650 5950 2950
+	5800 2125 5800 2200
 Wire Wire Line
-	5950 2950 5150 2950
-NoConn ~ 5050 2950
+	5800 2200 5650 2200
+$Comp
+L power:GND1 #PWR0103
+U 1 1 633E207F
+P 5350 2975
+F 0 "#PWR0103" H 5350 2725 50  0001 C CNN
+F 1 "GND1" H 5355 2802 50  0000 C CNN
+F 2 "" H 5350 2975 50  0001 C CNN
+F 3 "" H 5350 2975 50  0001 C CNN
+	1    5350 2975
+	1    0    0    -1
+$EndComp
 Wire Wire Line
-	5450 2650 5745 2650
-NoConn ~ 5450 2750
+	5350 2800 5350 2975
 $EndSCHEMATC

Commit message: smart-temp-only-sensor3
Parts:
- J1: footprint Connector_USB:USB_Mini-B_Tensility_54-00023_Vertical -> kicad3_footprint:USB_Mini-B_econ_connect_vertical
Connections:
- net GND1: now also J2.2 (Pin_2); no longer J2.4 (Pin_4)
- net SDA_GPIO_0: now reaches J1.2 (D-)
- net SDA_GPIO_0: now also J2.4 (Pin_4); no longer J2.3 (Pin_3)
- net SDL_GPIO_2: now reaches J1.3 (D+)
- net SDL_GPIO_2: now also J2.3 (Pin_3); no longer J2.2 (Pin_2)
Other:
- moved on the sheet: J2
Changed lines of the file:
@@
 L power:+3.3V #PWR0101
 U 1 1 633B9908
-P 6275 2150
-F 0 "#PWR0101" H 6275 2000 50  0001 C CNN
-F 1 "+3.3V" H 6290 2323 50  0000 C CNN
-F 2 "" H 6275 2150 50  0001 C CNN
-F 3 "" H 6275 2150 50  0001 C CNN
-	1    6275 2150
-	1    0    0    -1
+P 6425 2700
+F 0 "#PWR0101" H 6425 2550 50  0001 C CNN
+F 1 "+3.3V" H 6440 2873 50  0000 C CNN
+F 2 "" H 6425 2700 50  0001 C CNN
+F 3 "" H 6425 2700 50  0001 C CNN
+	1    6425 2700
+	-1   0    0    1
 $EndComp
 $Comp
 L power:GND1 #PWR0104
 U 1 1 633BE5C3
-P 6275 2775
-F 0 "#PWR0104" H 6275 2525 50  0001 C CNN
-F 1 "GND1" H 6280 2602 50  0000 C CNN
-F 2 "" H 6275 2775 50  0001 C CNN
-F 3 "" H 6275 2775 50  0001 C CNN
-	1    6275 2775
+P 6200 2700
+F 0 "#PWR0104" H 6200 2450 50  0001 C CNN
+F 1 "GND1" H 6205 2527 50  0000 C CNN
+F 2 "" H 6200 2700 50  0001 C CNN
+F 3 "" H 6200 2700 50  0001 C CNN
+	1    6200 2700
 	1    0    0    -1
 $EndComp
@@
 F 0 "J1" H 5407 2867 50  0000 C CNN
 F 1 "USB_B_Mini" H 5407 2776 50  0000 C CNN
-F 2 "Connector_USB:USB_Mini-B_Tensility_54-00023_Vertical" H 5500 2350 50  0001 C CNN
+F 2 "kicad3_footprint:USB_Mini-B_econ_connect_vertical" H 5500 2350 50  0001 C CNN
 F 3 "~" H 5500 2350 50  0001 C CNN
 	1    5350 2400
 	1    0    0    -1
 $EndComp
-$Comp
-L Connector:Conn_01x04_Female J2
-U 1 1 633D28B1
-P 6475 2400
-F 0 "J2" H 6503 2376 50  0000 L CNN
-F 1 "Conn_01x04_Female" H 6503 2285 50  0000 L CNN
-F 2 "Connector_PinSocket_2.54mm:PinSocket_1x04_P2.54mm_Vertical" H 6475 2400 50  0001 C CNN
-F 3 "~" H 6475 2400 50  0001 C CNN
-	1    6475 2400
-	1    0    0    -1
-$EndComp
-Wire Wire Line
-	6275 2300 6275 2150
-Wire Wire Line
-	6275 2400 5650 2400
-Wire Wire Line
-	5650 2500 6275 2500
-Wire Wire Line
-	6275 2600 6275 2775
 $Comp
 L power:+3.3V #PWR0102
@@
 	1    0    0    -1
 $EndComp
-Wire Wire Line
-	5800 2125 5800 2200
-Wire Wire Line
-	5800 2200 5650 2200
 $Comp
 L power:GND1 #PWR0103
@@
 Wire Wire Line
 	5350 2800 5350 2975
+$Comp
+L Connector:Conn_01x04_Female J2
+U 1 1 633D28B1
+P 6625 2400
+F 0 "J2" H 6653 2376 50  0000 L CNN
+F 1 "Conn_01x04_Female" H 6653 2285 50  0000 L CNN
+F 2 "Connector_PinSocket_2.54mm:PinSocket_1x04_P2.54mm_Vertical" H 6625 2400 50  0001 C CNN
+F 3 "~" H 6625 2400 50  0001 C CNN
+	1    6625 2400
+	1    0    0    1
+$EndComp
+Wire Wire Line
+	6425 2700 6425 2500
+Wire Wire Line
+	6200 2700 6200 2400
+Wire Wire Line
+	6200 2400 6425 2400
+Wire Wire Line
+	6425 2300 5650 2300
+Wire Wire Line
+	5650 2300 5650 2400
+Wire Wire Line
+	6425 2200 5925 2200
+Wire Wire Line
+	5925 2200 5925 2500
+Wire Wire Line
+	5925 2500 5650 2500
+Wire Wire Line
+	5650 2200 5800 2200
+Wire Wire Line
+	5800 2200 5800 2125
+Text Label 6000 2200 0    50   ~ 0
+SDA_GPIO_0
+Text Label 6000 2300 0    50   ~ 0
+SDL_GPIO_2
 $EndSCHEMATC

Commit message: double check conn
Connections:
- net SDA_GPIO_0: no longer names the net of J2.4 (Pin_4)
- net SDA_GPIO_0: now also J1.3 (D+); no longer J1.2 (D-)
- net SDL_GPIO_2 renamed SDL_GPIO_2-
- net SDL_GPIO_2-: now also J1.2 (D-); no longer J1.3 (D+)
Other:
- moved on the sheet: J2
Changed lines of the file:
@@
 L power:+3.3V #PWR0101
 U 1 1 633B9908
-P 6425 2700
-F 0 "#PWR0101" H 6425 2550 50  0001 C CNN
-F 1 "+3.3V" H 6440 2873 50  0000 C CNN
-F 2 "" H 6425 2700 50  0001 C CNN
-F 3 "" H 6425 2700 50  0001 C CNN
-	1    6425 2700
+P 6475 2900
+F 0 "#PWR0101" H 6475 2750 50  0001 C CNN
+F 1 "+3.3V" H 6490 3073 50  0000 C CNN
+F 2 "" H 6475 2900 50  0001 C CNN
+F 3 "" H 6475 2900 50  0001 C CNN
+	1    6475 2900
 	-1   0    0    1
 $EndComp
@@
 L power:GND1 #PWR0104
 U 1 1 633BE5C3
-P 6200 2700
-F 0 "#PWR0104" H 6200 2450 50  0001 C CNN
-F 1 "GND1" H 6205 2527 50  0000 C CNN
-F 2 "" H 6200 2700 50  0001 C CNN
-F 3 "" H 6200 2700 50  0001 C CNN
-	1    6200 2700
-	1    0    0    -1
-$EndComp
-$Comp
-L Connector:USB_B_Mini J1
-U 1 1 6339C102
-P 5350 2400
-F 0 "J1" H 5407 2867 50  0000 C CNN
-F 1 "USB_B_Mini" H 5407 2776 50  0000 C CNN
-F 2 "kicad3_footprint:USB_Mini-B_econ_connect_vertical" H 5500 2350 50  0001 C CNN
-F 3 "~" H 5500 2350 50  0001 C CNN
-	1    5350 2400
+P 6250 2900
+F 0 "#PWR0104" H 6250 2650 50  0001 C CNN
+F 1 "GND1" H 6255 2727 50  0000 C CNN
+F 2 "" H 6250 2900 50  0001 C CNN
+F 3 "" H 6250 2900 50  0001 C CNN
+	1    6250 2900
 	1    0    0    -1
 $EndComp
@@
 L Connector:Conn_01x04_Female J2
 U 1 1 633D28B1
-P 6625 2400
-F 0 "J2" H 6653 2376 50  0000 L CNN
-F 1 "Conn_01x04_Female" H 6653 2285 50  0000 L CNN
-F 2 "Connector_PinSocket_2.54mm:PinSocket_1x04_P2.54mm_Vertical" H 6625 2400 50  0001 C CNN
-F 3 "~" H 6625 2400 50  0001 C CNN
-	1    6625 2400
+P 6675 2600
+F 0 "J2" H 6703 2576 50  0000 L CNN
+F 1 "Conn_01x04_Female" H 6703 2485 50  0000 L CNN
+F 2 "Connector_PinSocket_2.54mm:PinSocket_1x04_P2.54mm_Vertical" H 6675 2600 50  0001 C CNN
+F 3 "~" H 6675 2600 50  0001 C CNN
+	1    6675 2600
 	1    0    0    1
 $EndComp
 Wire Wire Line
-	6425 2700 6425 2500
+	6475 2900 6475 2700
 Wire Wire Line
-	6200 2700 6200 2400
+	6250 2900 6250 2600
 Wire Wire Line
-	6200 2400 6425 2400
-Wire Wire Line
-	6425 2300 5650 2300
-Wire Wire Line
-	5650 2300 5650 2400
-Wire Wire Line
-	6425 2200 5925 2200
-Wire Wire Line
-	5925 2200 5925 2500
-Wire Wire Line
-	5925 2500 5650 2500
+	6250 2600 6475 2600
 Wire Wire Line
 	5650 2200 5800 2200
 Wire Wire Line
 	5800 2200 5800 2125
-Text Label 6000 2200 0    50   ~ 0
-SDA_GPIO_0
-Text Label 6000 2300 0    50   ~ 0
-SDL_GPIO_2
+Text Label 6025 2375 0    50   ~ 0
+SDA_GPIO_0+
+Text Label 6025 2500 0    50   ~ 0
+SDL_GPIO_2-
+$Comp
+L Connector:USB_B_Mini J1
+U 1 1 6339C102
+P 5350 2400
+F 0 "J1" H 5407 2867 50  0000 C CNN
+F 1 "USB_B_Mini" H 5407 2776 50  0000 C CNN
+F 2 "kicad3_footprint:USB_Mini-B_econ_connect_vertical" H 5500 2350 50  0001 C CNN
+F 3 "~" H 5500 2350 50  0001 C CNN
+	1    5350 2400
+	1    0    0    -1
+$EndComp
+Wire Wire Line
+	6475 2500 5650 2500
+Wire Wire Line
+	5650 2400 6475 2400
 $EndSCHEMATC
