File: kicad5/smart-temp-allinone/smart-temp-allinone.kicad_pcb (KiCad board)
At the start: 2 copper layers, 67.3 x 20.3 mm, 7 parts, among them J1 USB_A, J2 Conn_02x04_Odd_Even, J3 USB_A, J4 Conn_01x06_Female

Commit message: double check conn
Routing:
- net GND2: track 0.00 -> 59.7 mm
- net Net-(J2-Pad1): track 0.00 -> 57.1 mm
- net Net-(J2-Pad4): track 0.00 -> 52.3 mm
- net Net-(J2-Pad6): track 0.00 -> 52.3 mm
- net Net-(C1-Pad1): track 0.00 -> 32.5 mm
- net Net-(L1-Pad2): track 0.00 -> 14.6 mm
- net Net-(J3-Pad5): track 0.00 -> 13.1 mm
- net Net-(J1-Pad5): track 0.00 -> 13.1 mm
- net GND: track 0.00 -> 12.2 mm

Commit message: noid: add pwr
Parts:
- J4: footprint Connector_PinSocket_2.54mm:PinSocket_1x06_P2.54mm_Vertical -> Connector_PinSocket_2.54mm:PinSocket_1x06_P2.54mm_Horizontal
- moved J4 12.7 mm to (127.8, 80.0), turned to 0 degrees
- moved C1 2.47 mm to (85.6, 81.5), turned to 90 degrees
- moved J3 1.55 mm to (133.1, 90.1)
- moved J2 0.62 mm to (87.0, 85.3)
- moved PS1 0.55 mm to (90.7, 82.8)
- moved J1 0.52 mm to (79.4, 82.9)
- moved L1 0.09 mm to (102.9, 82.9)
Connections:
- net Net-(C1-Pad1) renamed +5V
- net Net-(J2-Pad1) renamed +3V3
Routing:
- net +3V3: track 57.1 -> 72.9 mm
- net Net-(J2-Pad6): track 52.3 -> 58.8 mm
- net GND2: track 59.7 -> 54.1 mm
- net GND: track 12.2 -> 15.1 mm
- net +5V: track 32.5 -> 29.7 mm
- net Net-(J2-Pad4): track 52.3 -> 50.8 mm
- net Net-(L1-Pad2): track 14.6 -> 14.1 mm

Commit message: noid: update
Parts:
- J4: footprint Connector_PinSocket_2.54mm:PinSocket_1x06_P2.54mm_Horizontal -> Connector_PinSocket_2.54mm:PinSocket_1x06_P2.54mm_Vertical
- moved J4 12.7 mm to (128.2, 92.7), turned to 180 degrees
- moved J2 7.94 mm to (84.5, 92.9), turned to 180 degrees
Routing:
- net +3V3: track 72.9 -> 57.4 mm
- net Net-(J2-Pad6): track 58.8 -> 46.9 mm
- net Net-(J2-Pad4): track 50.8 -> 49.5 mm
- net Net-(J1-Pad5): track 13.1 -> 14.1 mm
- net GND2: track 54.1 -> 53.2 mm
Other:
- outline, holes or cut-outs redrawn
